Commit message: Finger joits -> static

File: UR5e/BrainCoRightHandURDF/urdf/BrainCoRightHandURDF.urdf.xacro (robot description, xacro)
@@ -87,5 +87,5 @@
     <joint
       name="${prefix}thumbCMC"
-      type="revolute">
+      type="fixed">
       <origin
         xyz="0.0245 0.0242 0.021628"
@@ -95,11 +95,4 @@
       <child
         link="${prefix}thumb_prox" />
-      <axis
-        xyz="0 -1 0" />
-      <limit
-        lower="0"
-        upper="1.5708"
-        effort="0"
-        velocity="0" />
     </joint>
     <link
@@ -145,5 +138,5 @@
     <joint
       name="${prefix}thumbMCP"
-      type="revolute">
+      type="fixed">
       <origin
         xyz="0.013647 0 0"
@@ -153,11 +146,4 @@
       <child
         link="${prefix}thumb_dist" />
-      <axis
-        xyz="0 0 1" />
-      <limit
-        lower="0"
-        upper="0.87266"
-        effort="0"
-        velocity="0" />
     </joint>
     <link
@@ -203,5 +189,5 @@
     <joint
       name="${prefix}indexMCP"
-      type="revolute">
+      type="fixed">
       <origin
         xyz="0.029003 0.088231 -0.0039488"
@@ -211,11 +197,4 @@
       <child
         link="${prefix}index_prox" />
-      <axis
-        xyz="1 0 0" />
-      <limit
-        lower="0"
-        upper="1.309"
-        effort="0"
-        velocity="0" />
     </joint>
     <link
@@ -261,5 +240,5 @@
     <joint
       name="${prefix}indexPIP"
-      type="revolute">
+      type="fixed">
       <origin
         xyz="0 0.035 0"
@@ -269,11 +248,4 @@
       <child
         link="${prefix}index_dist" />
-      <axis
-        xyz="1 0 0" />
-      <limit
-        lower="0"
-        upper="2.0944"
-        effort="0"
-        velocity="0" />
     </joint>
     <link
@@ -319,5 +291,5 @@
     <joint
       name="${prefix}middleMCP"
-      type="revolute">
+      type="fixed">
       <origin
         xyz="0.008 0.091935 -0.0082038"
@@ -327,11 +299,4 @@
       <child
         link="${prefix}middle_prox" />
-      <axis
-        xyz="1 0 0" />
-      <limit
-        lower="0"
-        upper="1.309"
-        effort="0"
-        velocity="0" />
     </joint>
     <link
@@ -377,5 +342,5 @@
     <joint
       name="${prefix}middlePIP"
-      type="revolute">
+      type="fixed">
       <origin
         xyz="0 0.042 0"
@@ -385,11 +350,4 @@
       <child
         link="${prefix}middle_dist" />
-      <axis
-        xyz="1 0 0" />
-      <limit
-        lower="0"
-        upper="2.0944"
-        effort="0"
-        velocity="0" />
     </joint>
     <link
@@ -435,5 +393,5 @@
     <joint
       name="${prefix}ringMCP"
-      type="revolute">
+      type="fixed">
       <origin
         xyz="-0.013103 0.089947 -0.0080786"
@@ -443,11 +401,4 @@
       <child
         link="${prefix}ring_prox" />
-      <axis
-        xyz="1 0 0" />
-      <limit
-        lower="0"
-        upper="1.309"
-        effort="0"
-        velocity="0" />
     </joint>
     <link
@@ -493,5 +444,5 @@
     <joint
       name="${prefix}ringPIP"
-      type="revolute">
+      type="fixed">
       <origin
         xyz="0 0.042 0"
@@ -501,11 +452,4 @@
       <child
         link="${prefix}ring_dist" />
-      <axis
-        xyz="1 0 0" />
-      <limit
-        lower="0"
-        upper="2.0944"
-        effort="0"
-        velocity="0" />
     </joint>
     <link
@@ -551,5 +495,5 @@
     <joint
       name="${prefix}littleMCP"
-      type="revolute">
+      type="fixed">
       <origin
         xyz="-0.033731 0.083727 -0.0036339"
@@ -559,11 +503,4 @@
       <child
         link="${prefix}little_prox" />
-      <axis
-        xyz="1 0 0" />
-      <limit
-        lower="0"
-        upper="1.309"
-        effort="0"
-        velocity="0" />
     </joint>
     <link
@@ -609,5 +546,5 @@
     <joint
       name="${prefix}littlePIP"
-      type="revolute">
+      type="fixed">
       <origin
         xyz="0 0.035 0"
@@ -617,11 +554,4 @@
       <child
         link="${prefix}little_dist" />
-      <axis
-        xyz="1 0 0" />
-      <limit
-        lower="0"
-        upper="2.0944"
-        effort="0"
-        velocity="0" />
     </joint>
   </xacro:macro>

Commit message: UR5e files cleanup

File: UR5e/BrainCoRightHandURDF/urdf/BrainCoRightHandURDF.urdf.xacro (robot description, xacro)
@@ -1,557 +1,299 @@
-<?xml version="1.0" encoding="utf-8"?>
+<?xml version="1.0" ?>
 <!-- This URDF was automatically created by SolidWorks to URDF Exporter! Originally created by Stephen Brawner (brawner@gmail.com)
      Commit Version: 1.6.0-4-g7f85cfe  Build Version: 1.6.7995.38578
      For more information, please see http://wiki.ros.org/sw_urdf_exporter -->
-<robot name="BrainCoRightHandURDF" xmlns:xacro="http://wiki.ros.org/xacro">
+<robot xmlns:xacro="http://wiki.ros.org/xacro" name="BrainCoRightHandURDF">
   <xacro:macro name="brainco_hand" params="prefix:=''">
-    <link
-      name="${prefix}base_link">
-      <inertial>
-        <origin
-          xyz="-0.00099373 0.040537 -0.0022835"
-          rpy="0 0 0" />
-        <mass
-          value="0.427" />
-        <inertia
-          ixx="3.4364E-05"
-          ixy="-1.2404E-06"
-          ixz="5.654E-07"
-          iyy="3.9467E-05"
-          iyz="3.8955E-06"
-          izz="6.3984E-05" />
-      </inertial>
-      <visual>
-        <origin
-          xyz="0 0 0"
-          rpy="0 0 0" />
-        <geometry>
-          <mesh
-            filename="package://BrainCoRightHandURDF/meshes/base_link.STL" />
-        </geometry>
-        <material
-          name="">
-          <color
-            rgba="0.75294 0.75294 0.75294 1" />
-        </material>
-      </visual>
-      <collision>
-        <origin
-          xyz="0 0 0"
-          rpy="0 0 0" />
-        <geometry>
-          <mesh
-            filename="package://BrainCoRightHandURDF/meshes/base_link.STL" />
-        </geometry>
-      </collision>
-    </link>
-    <link
-      name="${prefix}thumb_prox">
-      <inertial>
-        <origin
-          xyz="0.0062041 -7.9383E-08 0.0015306"
-          rpy="0 0 0" />
-        <mass
-          value="0.005" />
-        <inertia
-          ixx="4.0639E-08"
-          ixy="5.8675E-13"
-          ixz="2.4299E-09"
-          iyy="9.2485E-08"
-          iyz="7.1049E-13"
-          izz="8.5586E-08" />
-      </inertial>
-      <visual>
-        <origin
-          xyz="0 0 0"
-          rpy="0 0 0" />
-        <geometry>
-          <mesh
-            filename="package://BrainCoRightHandURDF/meshes/thumb_prox.STL" />
-        </geometry>
-        <material
-          name="">
-          <color
-            rgba="1 1 1 1" />
-        </material>
-      </visual>
-      <collision>
-        <origin
-          xyz="0 0 0"
-          rpy="0 0 0" />
-        <geometry>
-          <mesh
-            filename="package://BrainCoRightHandURDF/meshes/thumb_prox.STL" />
-        </geometry>
-      </collision>
-    </link>
-    <joint
-      name="${prefix}thumbCMC"
-      type="fixed">
-      <origin
-        xyz="0.0245 0.0242 0.021628"
-        rpy="0 -0.49642 0" />
-      <parent
-        link="${prefix}base_link" />
-      <child
-        link="${prefix}thumb_prox" />
-    </joint>
-    <link
-      name="${prefix}thumb_dist">
-      <inertial>
-        <origin
-          xyz="0.0083564 0.037204 -3.5884E-07"
-          rpy="0 0 0" />
-        <mass
-          value="0.04" />
-        <inertia
-          ixx="7.1498E-06"
-          ixy="2.0157E-07"
-          ixz="-6.0726E-11"
-          iyy="9.1501E-07"
-          iyz="5.4502E-10"
-          izz="6.8747E-06" />
-      </inertial>
-      <visual>
-        <origin
-          xyz="0 0 0"
-          rpy="0 0 0" />
-        <geometry>
-          <mesh
-            filename="package://BrainCoRightHandURDF/meshes/thumb_dist.STL" />
-        </geometry>
-        <material
-          name="">
-          <color
-            rgba="0.75294 0.75294 0.75294 1" />
-        </material>
-      </visual>
-      <collision>
-        <origin
-          xyz="0 0 0"
-          rpy="0 0 0" />
-        <geometry>
-          <mesh
-            filename="package://BrainCoRightHandURDF/meshes/thumb_dist.STL" />
-        </geometry>
-      </collision>
-    </link>
-    <joint
-      name="${prefix}thumbMCP"
-      type="fixed">
-      <origin
-        xyz="0.013647 0 0"
-        rpy="-0.39332 0.31115 -0.93514" />
-      <parent
-        link="${prefix}thumb_prox" />
-      <child
-        link="${prefix}thumb_dist" />
-    </joint>
-    <link
-      name="${prefix}index_prox">
-      <inertial>
-        <origin
-          xyz="-5.571E-07 0.016609 0.00045746"
-          rpy="0 0 0" />
-        <mass
-          value="0.008" />
-        <inertia
-          ixx="3.3526E-07"
-          ixy="2.9401E-11"
-          ixz="-2.4782E-12"
-          iyy="1.0133E-07"
-          iyz="2.0576E-08"
-          izz="3.7092E-07" />
-      </inertial>
-      <visual>
-        <origin
-          xyz="0 0 0"
-          rpy="0 0 0" />
-        <geometry>
-          <mesh
-            filename="package://BrainCoRightHandURDF/meshes/index_prox.STL" />
-        </geometry>
-        <material
-          name="">
-          <color
-            rgba="0.75294 0.75294 0.75294 1" />
-        </material>
-      </visual>
-      <collision>
-        <origin
-          xyz="0 0 0"
-          rpy="0 0 0" />
-        <geometry>
-          <mesh
-            filename="package://BrainCoRightHandURDF/meshes/index_prox.STL" />
-        </geometry>
-      </collision>
-    </link>
-    <joint
-      name="${prefix}indexMCP"
-      type="fixed">
-      <origin
-        xyz="0.029003 0.088231 -0.0039488"
-        rpy="-0.09929 -0.054667 -0.031168" />
-      <parent
-        link="${prefix}base_link" />
-      <child
-        link="${prefix}index_prox" />
-    </joint>
-    <link
-      name="${prefix}index_dist">
-      <inertial>
-        <origin
-          xyz="5.9401E-06 0.025449 0.003278"
-          rpy="0 0 0" />
-        <mass
-          value="0.011" />
-        <inertia
-          ixx="8.4801E-07"
-          ixy="-1.0878E-09"
-          ixz="-1.3683E-10"
-          iyy="1.4147E-07"
-          iyz="-1.0078E-07"
-          izz="8.5502E-07" />
-      </inertial>
-      <visual>
-        <origin
-          xyz="0 0 0"
-          rpy="0 0 0" />
-        <geometry>
-          <mesh
-            filename="package://BrainCoRightHandURDF/meshes/index_dist.STL" />
-        </geometry>
-        <material
-          name="">
-          <color
-            rgba="0.75294 0.75294 0.75294 1" />
-        </material>
-      </visual>
-      <collision>
-        <origin
-          xyz="0 0 0"
-          rpy="0 0 0" />
-        <geometry>
-          <mesh
-            filename="package://BrainCoRightHandURDF/meshes/index_dist.STL" />
-        </geometry>
-      </collision>
-    </link>
-    <joint
-      name="${prefix}indexPIP"
-      type="fixed">
-      <origin
-        xyz="0 0.035 0"
-        rpy="0.19353 0 0" />
-      <parent
-        link="${prefix}index_prox" />
-      <child
-        link="${prefix}index_dist" />
-    </joint>
-    <link
-      name="${prefix}middle_prox">
-      <inertial>
-        <origin
-          xyz="2.3779E-07 0.020205 0.00053993"
-          rpy="0 0 0" />
-        <mass
-          value="0.011" />
-        <inertia
-          ixx="5.5624E-07"
-          ixy="8E-12"
-          ixz="-8.5151E-12"
-          iyy="1.3298E-07"
-          iyz="2.669E-08"
-          izz="6.0146E-07" />
-      </inertial>
-      <visual>
-        <origin
-          xyz="0 0 0"
-          rpy="0 0 0" />
-        <geometry>
-          <mesh
-            filename="package://BrainCoRightHandURDF/meshes/middle_prox.STL" />
-        </geometry>
-        <material
-          name="">
-          <color
-            rgba="0.75294 0.75294 0.75294 1" />
-        </material>
-      </visual>
-      <collision>
-        <origin
-          xyz="0 0 0"
-          rpy="0 0 0" />
-        <geometry>
-          <mesh
-            filename="package://BrainCoRightHandURDF/meshes/middle_prox.STL" />
-        </geometry>
-      </collision>
-    </link>
-    <joint
-      name="${prefix}middleMCP"
-      type="fixed">
-      <origin
-        xyz="0.008 0.091935 -0.0082038"
-        rpy="-0.069813 0 0" />
-      <parent
-        link="${prefix}base_link" />
-      <child
-        link="${prefix}middle_prox" />
-    </joint>
-    <link
-      name="${prefix}middle_dist">
-      <inertial>
-        <origin
-          xyz="5.9404E-06 0.025449 0.003278"
-          rpy="0 0 0" />
-        <mass
-          value="0.011" />
-        <inertia
-          ixx="8.4801E-07"
-          ixy="-1.0879E-09"
-          ixz="-1.3705E-10"
-          iyy="1.4147E-07"
-          iyz="-1.0078E-07"
-          izz="8.5501E-07" />
-      </inertial>
-      <visual>
-        <origin
-          xyz="0 0 0"
-          rpy="0 0 0" />
-        <geometry>
-          <mesh
-            filename="package://BrainCoRightHandURDF/meshes/middle_dist.STL" />
-        </geometry>
-        <material
-          name="">
-          <color
-            rgba="0.75294 0.75294 0.75294 1" />
-        </material>
-      </visual>
-      <collision>
-        <origin
-          xyz="0 0 0"
-          rpy="0 0 0" />
-        <geometry>
-          <mesh
-            filename="package://BrainCoRightHandURDF/meshes/middle_dist.STL" />
-        </geometry>
-      </collision>
-    </link>
-    <joint
-      name="${prefix}middlePIP"
-      type="fixed">
-      <origin
-        xyz="0 0.042 0"
-        rpy="0.18357 0 0" />
-      <parent
-        link="${prefix}middle_prox" />
-      <child
-        link="${prefix}middle_dist" />
-    </joint>
-    <link
-      name="${prefix}ring_prox">
-      <inertial>
-        <origin
-          xyz="2.4507E-07 0.020236 0.00042373"
-          rpy="0 0 0" />
-        <mass
-          value="0.011" />
-        <inertia
-          ixx="5.5623E-07"
-          ixy="7.4604E-12"
-          ixz="-8.5876E-12"
-          iyy="1.3295E-07"
-          iyz="2.7719E-08"
-          izz="6.0149E-07" />
-      </inertial>
-      <visual>
-        <origin
-          xyz="0 0 0"
-          rpy="0 0 0" />
-        <geometry>
-          <mesh
-            filename="package://BrainCoRightHandURDF/meshes/ring_prox.STL" />
-        </geometry>
-        <material
-          name="">
-          <color
-            rgba="0.75294 0.75294 0.75294 1" />
-        </material>
-      </visual>
-      <collision>
-        <origin
-          xyz="0 0 0"
-          rpy="0 0 0" />
-        <geometry>
-          <mesh
-            filename="package://BrainCoRightHandURDF/meshes/ring_prox.STL" />
-        </geometry>
-      </collision>
-    </link>
-    <joint
-      name="${prefix}ringMCP"
-      type="fixed">
-      <origin
-        xyz="-0.013103 0.089947 -0.0080786"
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