Commit message: UR5e files cleanup

File: UR5e/duo_ur/urdf/duo_ur_onehand.urdf.xacro (robot description, xacro)
@@ -1,16 +1,8 @@
 <?xml version="1.0"?>
-<!-- <xacro:arg name="name" default="ur"/> -->
-<!-- <robot xmlns:xacro="http://wiki.ros.org/xacro" name="$(arg name)"> -->
 <robot xmlns:xacro="http://wiki.ros.org/xacro" name="ur">
-   <!-- robot name parameter -->
    <xacro:arg name="name" default="ur"/>
-   <!-- import main macro -->
    <xacro:include filename="$(find duo_ur)/urdf/ur5e_macro.xacro"/>
    <xacro:include filename="$(find BrainCoRightHandURDF)/urdf/BrainCoRightHandURDF.urdf.xacro"/>
-   <!-- possible 'ur_type' values ur3, ur3e, ur5, ur5e, ur7e, ur10, ur10e, ur12e, ur16e, ur20, ur30 -->
-   <!-- the default value should raise an error in case this was called without defining the type -->
    <xacro:arg name="ur_type" default="ur5e"/>
-   <!-- parameters -->
-   <!-- <xacro:arg name="tf_prefix" default="" /> -->
    <xacro:arg name="tf_prefix_1" default="right_" />
    <xacro:arg name="tf_prefix_2" default="left_" />
@@ -23,5 +15,4 @@
    <xacro:arg name="safety_pos_margin" default="0.15"/>
    <xacro:arg name="safety_k_position" default="20"/>
-   <!-- ros2_control related parameters -->
    <xacro:arg name="headless_mode" default="false" />
    <xacro:arg name="robot_ip_1" default="192.168.1.102" />
@@ -39,5 +30,4 @@
    <xacro:arg name="script_sender_port_2" default="50012"/>
    <xacro:arg name="trajectory_port_2" default="50013"/>
-   <!--   tool communication related parameters-->
    <xacro:arg name="use_tool_communication" default="false" />
    <xacro:arg name="tool_voltage" default="0" />
@@ -49,18 +39,14 @@
    <xacro:arg name="tool_device_name" default="/tmp/ttyUR" />
    <xacro:arg name="tool_tcp_port" default="54321" />
-     <!-- Simulation parameters -->
-   <xacro:arg name="use_fake_hardware" default="true" /> <!-- #### -->
+   <xacro:arg name="use_fake_hardware" default="true" />
    <xacro:arg name="fake_sensor_commands" default="false" />
    <xacro:arg name="sim_gazebo" default="false" />
    <xacro:arg name="sim_ignition" default="false" />
    <xacro:arg name="simulation_controllers" default="$(find duo_ur)/config/duo_ur5e_controllers.yaml" />
-   <!-- <xacro:arg name="simulation_controllers" default="$(find duo_ur_moveit_config)/config/ros2_controllers.yaml" /> -->
    <material name="Light_Grey">
     <color rgba="0.8 0.8 0.8 1.0"/>
   </material>
-   <!-- initial position for simulations (Fake Hardware, Gazebo, Ignition) -->
    <xacro:arg name="initial_positions_file_1" default="$(find duo_ur)/config/$(arg tf_prefix_1)initial_positions.yaml"/>
    <xacro:arg name="initial_positions_file_2" default="$(find duo_ur)/config/$(arg tf_prefix_2)initial_positions.yaml"/>
-   <!-- convert to property to use substitution in function -->
    <xacro:property name="initial_positions_file_1" default="$(arg initial_positions_file_1)"/>
    <xacro:property name="initial_positions_file_2" default="$(arg initial_positions_file_2)"/>
@@ -78,27 +64,12 @@
    <xacro:property name="plate_dimension" value="0.18 0.18 0.02"/>
    <xacro:property name="left_plate_origin" value="0 -0.16 0.01807"/>
-   <xacro:property name="right_plate_origin" value="0 0.16 0.025"/> <!-- TODO change -->
+   <xacro:property name="right_plate_origin" value="0 0.16 0.025"/>
    <xacro:property name="base_mount_origin" value="0 0 0.01"/>
    <xacro:property name="camera_base_radius" value="0.0375"/>
    <xacro:property name="camera_base_length" value="0.025"/>
    <xacro:property name="camera_base_origin" value="0 0 0.007"/>
-   <xacro:property name="camera_shaft_dimension" value="0.11 0.022 0.016"/>
-   <xacro:property name="camera_shaft_origin" value="0.07 0 -0.0045"/>
-   <xacro:property name="camera_dimension" value="0.06 0.13 0.03"/>
-   <xacro:property name="camera_origin" value="0.055 0 0.02"/>
-   <!-- <xacro:property name="camera_rotation" value="3.14159265359 -1.570796 0"/> -->
-   <xacro:property name="camera_rotation" value="3.14159265359 -1.570796 0"/>
-   <!-- <xacro:property name="camera_link_origin" value="0 0 -0.013624"/> -->
-   <xacro:property name="camera_link_origin" value="0.025 0.0475 0"/>
-   <!-- <xacro:property name="camera_rotation" value="0 0 1.570796"/> -->
    <xacro:property name="sensor_base_radius" value="0.0575"/>
    <xacro:property name="sensor_base_length" value="0.035"/>
    <xacro:property name="sensor_base_origin" value="0 0 0.03"/>
-   <xacro:property name="pruner_base_radius" value="0.05"/>
-   <xacro:property name="pruner_base_length" value="0.3"/>
-   <xacro:property name="pruner_base_origin" value="0 0 0.1675"/>
-   <xacro:property name="tcp_origin" value="0 0 0.15"/>
-   <!-- <xacro:property name="tcp_origin" value="0 0 0.32"/> -->
-   <!-- create link fixed to the "world" -->
    <link name="world" />
   <link name="mur">
@@ -190,5 +161,5 @@
     <parent link="torso"/>
     <child link="chest"/>
-    <origin xyz="0.1 0 0" rpy="0 0 0"/>  <!-- tune this to where you want "chest" to be -->
+    <origin xyz="0.1 0 0" rpy="0 0 0"/>
   </joint>
   <link name="$(arg tf_prefix_1)plate">
@@ -212,7 +183,4 @@
     <child link="$(arg tf_prefix_1)plate"/>
     <origin xyz="${left_plate_origin}" rpy="2.35619449019 0 0"/>
-    <!-- Here we define the axis along which the geometry is moved -->
-    <!-- <axis xyz="0 1 0"/> -->
-    <!-- Here we define the joint's upper and lower limits -->
     <limit effort="1000.0" lower="-0.5" upper="0.5" velocity="0.5"/>
   </joint>
@@ -222,7 +190,5 @@
     <child link="$(arg tf_prefix_1)base_mount"/>
     <origin xyz="${base_mount_origin}" rpy="0 0 -0.0127409035"/>
-    <!-- Here we define the axis along which the geometry is moved -->
     <axis xyz="0 0 0"/>
-    <!-- Here we define the joint's upper and lower limits -->
     <limit effort="1000.0" lower="-0.5" upper="0.5" velocity="0.5"/>
   </joint>
@@ -247,7 +213,4 @@
     <child link="$(arg tf_prefix_2)plate"/>
     <origin xyz="${right_plate_origin}" rpy="2.35619449019 0 3.14159265359"/>
-    <!-- Here we define the axis along which the geometry is moved -->
-    <!-- <axis xyz="0 1 0"/> -->
-    <!-- Here we define the joint's upper and lower limits -->
     <limit effort="1000.0" lower="-0.5" upper="0.5" velocity="0.5"/>
   </joint>
@@ -256,8 +219,6 @@
     <parent link="$(arg tf_prefix_2)plate"/>
     <child link="$(arg tf_prefix_2)base_mount"/>
-    <origin xyz="${base_mount_origin}"/> <!-- TODO calibrate right hand rotation -->
-    <!-- Here we define the axis along which the geometry is moved -->
+    <origin xyz="${base_mount_origin}"/>
     <axis xyz="0 0 0"/>
-    <!-- Here we define the joint's upper and lower limits -->
     <limit effort="1000.0" lower="-0.5" upper="0.5" velocity="0.5"/>
   </joint>
@@ -286,5 +247,4 @@
      </joint>
    </xacro:if>
-   <!-- arm_1 -->
    <xacro:ur_robot
      name="$(arg tf_prefix_1)$(arg name)"
@@ -324,5 +284,5 @@
      trajectory_port="$(arg trajectory_port_1)"
      >
-     <origin xyz="0 0 0" rpy="0 0 0" />          <!-- position robot in the world -->
+     <origin xyz="0 0 0" rpy="0 0 0" />
    </xacro:ur_robot>
    <link name="$(arg tf_prefix_1)camera_base">
@@ -347,52 +307,4 @@
     <origin xyz="${camera_base_origin}" rpy="0 0 0"/>
   </joint>
-  <!-- <link name="$(arg tf_prefix_1)camera_shaft">
-    <visual>
-      <geometry>
-        <box size="${camera_shaft_dimension}"/>
-      </geometry>
-      <origin rpy="0 0 0" xyz="0 0 0"/>
-      <material name="red">
-        <color rgba="0.8 0 0 .6"/>
-      </material>
-    </visual>
-    <collision>
-      <geometry>
-        <box size="${camera_shaft_dimension}"/>
-      </geometry>
-    </collision>
-  </link>
-  <joint name="$(arg tf_prefix_1)camera_base_to_camera_shaft" type="fixed">
-    <parent link="$(arg tf_prefix_1)camera_base"/>
-    <child link="$(arg tf_prefix_1)camera_shaft"/>
-    <origin xyz="${camera_shaft_origin}" rpy="0 0 0"/>
-  </joint>
-  <link name="$(arg tf_prefix_1)camera">
-    <visual>
-      <geometry>
-        <box size="${camera_dimension}"/>
-      </geometry>
-      <origin rpy="0 0 0" xyz="0 0 0"/>
-      <material name="blue">
-        <color rgba="0 0 0.8 .6"/>
-      </material>
-    </visual>
-    <collision>
-      <geometry>
-        <box size="${camera_dimension}"/>
-      </geometry>
-    </collision>
-  </link>
-  <joint name="$(arg tf_prefix_1)camera_shaft_to_camera" type="fixed">
-    <parent link="$(arg tf_prefix_1)camera_shaft"/>
-    <child link="$(arg tf_prefix_1)camera"/>
-    <origin xyz="${camera_origin}" rpy="${camera_rotation}"/>
-  </joint>
-  <link name="$(arg tf_prefix_1)camera_link"/>
-  <joint name="$(arg tf_prefix_1)camera_to_camera_link" type="fixed">
-    <parent link="$(arg tf_prefix_1)camera"/>
-    <child link="$(arg tf_prefix_1)camera_link"/>
-    <origin xyz="${camera_link_origin}" rpy="0 0 0"/>
-  </joint> -->
   <link name="$(arg tf_prefix_1)sensor_base">
     <visual>
@@ -441,42 +353,10 @@
     <origin xyz="0 0 0.0487" rpy="1.5708 0 -2.0943951"/>
   </joint>
-  <!-- <origin xyz="0 0 0.0487" rpy="1.5708 0 -1.04721"/> -->
-  <!-- <origin xyz="0 0 0.0487" rpy="1.5708 0 -1.5708"/> -->
   <link name="$(arg tf_prefix_1)tcp"/>
-  <joint name="$(arg tf_prefix_1)pruner_base_to_tcp" type="fixed">
+  <joint name="$(arg tf_prefix_1)hand_base_to_tcp" type="fixed">
     <parent link="$(arg tf_prefix_1)hand_base_link"/>
     <child link="$(arg tf_prefix_1)tcp"/>
-    <origin xyz="0 0.028 -0.01" rpy="0 3.1416 -1.5708"/> <!-- 0.028 -->
-  </joint>
-  <!--
-  <link name="$(arg tf_prefix_1)pruner_base">
-    <visual>
-      <geometry>
-        <cylinder length="${pruner_base_length}" radius="${pruner_base_radius}"/>
-      </geometry>
-      <origin rpy="0 0 0" xyz="0 0 0"/>
-      <material name="green">
-        <color rgba="0 0.8 0 .6"/>
-      </material>
-    </visual>
-    <collision>
-      <geometry>
-        <cylinder length="${pruner_base_length}" radius="${pruner_base_radius}"/>
-      </geometry>
-    </collision>
-  </link>
-  <joint name="$(arg tf_prefix_1)sensor_base_to_pruner_base" type="fixed">
-    <parent link="$(arg tf_prefix_1)sensor_base"/>
-    <child link="$(arg tf_prefix_1)pruner_base"/>
-    <origin xyz="${pruner_base_origin}" rpy="0 0 0"/>
-  </joint>
-  <link name="$(arg tf_prefix_1)tcp"/>
-  <joint name="$(arg tf_prefix_1)pruner_base_to_tcp" type="fixed">
-    <parent link="$(arg tf_prefix_1)pruner_base"/>
-    <child link="$(arg tf_prefix_1)tcp"/>
-    <origin xyz="${tcp_origin}" rpy="0 0 0"/>
-  </joint>
-  -->
-  <!-- arm_2 -->
+    <origin xyz="0 0.028 -0.01" rpy="0 3.1416 -1.5708"/>
+  </joint>
    <xacro:ur_robot
      name="$(arg tf_prefix_2)$(arg name)"
@@ -516,5 +396,5 @@
      trajectory_port="$(arg trajectory_port_2)"
      >
-     <origin xyz="0 0 0" rpy="0 0 0" />          <!-- position robot in the world -->
+     <origin xyz="0 0 0" rpy="0 0 0" />
    </xacro:ur_robot>
    <link name="$(arg tf_prefix_2)camera_base">
@@ -539,52 +419,4 @@
     <origin xyz="${camera_base_origin}" rpy="0 0 0"/>
   </joint>
-  <!-- <link name="$(arg tf_prefix_2)camera_shaft">
-    <visual>
-      <geometry>
-        <box size="${camera_shaft_dimension}"/>
-      </geometry>
-      <origin rpy="0 0 0" xyz="0 0 0"/>
-      <material name="red">
-        <color rgba="0.8 0 0 .6"/>
-      </material>
-    </visual>
-    <collision>
-      <geometry>
-        <box size="${camera_shaft_dimension}"/>
-      </geometry>
-    </collision>
-  </link>
-  <joint name="$(arg tf_prefix_2)camera_base_to_camera_shaft" type="fixed">
-    <parent link="$(arg tf_prefix_2)camera_base"/>
-    <child link="$(arg tf_prefix_2)camera_shaft"/>
-    <origin xyz="${camera_shaft_origin}" rpy="0 0 0"/>
-  </joint>
-  <link name="$(arg tf_prefix_2)camera">
-    <visual>
-      <geometry>
-        <box size="${camera_dimension}"/>
-      </geometry>
-      <origin rpy="0 0 0" xyz="0 0 0"/>
-      <material name="blue">
-        <color rgba="0 0 0.8 .6"/>
-      </material>
-    </visual>
-    <collision>
-      <geometry>
-        <box size="${camera_dimension}"/>
-      </geometry>
-    </collision>
-  </link>
-  <joint name="$(arg tf_prefix_2)camera_shaft_to_camera" type="fixed">
-    <parent link="$(arg tf_prefix_2)camera_shaft"/>
-    <child link="$(arg tf_prefix_2)camera"/>
-    <origin xyz="${camera_origin}" rpy="${camera_rotation}"/>
-  </joint>
-  <link name="$(arg tf_prefix_2)camera_link"/>
-  <joint name="$(arg tf_prefix_2)camera_to_camera_link" type="fixed">
-    <parent link="$(arg tf_prefix_2)camera"/>
-    <child link="$(arg tf_prefix_2)camera_link"/>
-    <origin xyz="${camera_link_origin}" rpy="0 0 0"/>
-  </joint> -->
   <link name="$(arg tf_prefix_2)sensor_base">
     <visual>
@@ -608,31 +440,4 @@
     <origin xyz="${sensor_base_origin}" rpy="0 0 0"/>
   </joint>
-  <!--link name="$(arg tf_prefix_2)pruner_base">
-    <visual>
-      <geometry>
-        <cylinder length="${pruner_base_length}" radius="${pruner_base_radius}"/>
-      </geometry>
-      <origin rpy="0 0 0" xyz="0 0 0"/>
-      <material name="green">
-        <color rgba="0 0.8 0 .6"/>
-      </material>
-    </visual>
-    <collision>
-      <geometry>
-        <cylinder length="${pruner_base_length}" radius="${pruner_base_radius}"/>
-      </geometry>
-    </collision>
-  </link>
-  <joint name="$(arg tf_prefix_2)sensor_base_to_pruner_base" type="fixed">
-    <parent link="$(arg tf_prefix_2)sensor_base"/>
-    <child link="$(arg tf_prefix_2)pruner_base"/>
-    <origin xyz="${pruner_base_origin}" rpy="0 0 0"/>
-  </joint>
-  <link name="$(arg tf_prefix_2)tcp"/>
-  <joint name="$(arg tf_prefix_2)pruner_base_to_tcp" type="fixed">
-    <parent link="$(arg tf_prefix_2)pruner_base"/>
-    <child link="$(arg tf_prefix_2)tcp"/>
-    <origin xyz="${tcp_origin}" rpy="0 0 0"/>
-  </joint-->
   <link name="$(arg tf_prefix_2)hand_connector_link">
     <visual>
@@ -660,14 +465,11 @@
     <origin xyz="0 0 0.0487" rpy="1.5708 0 -2.0943951"/>
   </joint>
-  <!-- <origin xyz="0 0 0.0487" rpy="1.5708 0 -1.04721"/> -->
-  <!-- <origin xyz="0 0 0.0487" rpy="1.5708 0 -1.5708"/> -->
   <link name="$(arg tf_prefix_2)tcp"/>
-  <joint name="$(arg tf_prefix_2)pruner_base_to_tcp" type="fixed">
+  <joint name="$(arg tf_prefix_2)hand_base_to_tcp" type="fixed">
     <parent link="$(arg tf_prefix_2)hand_base_link"/>
     <child link="$(arg tf_prefix_2)tcp"/>
-    <origin xyz="0 0.028 -0.01" rpy="0 3.1416 -1.5708"/> <!-- 0.028 -->
+    <origin xyz="0 0.028 -0.01" rpy="0 3.1416 -1.5708"/>
   </joint>
    <xacro:if value="$(arg sim_gazebo)">
-    <!-- Gazebo plugins -->
     <gazebo reference="world">
     </gazebo>
@@ -679,5 +481,4 @@
   </xacro:if>
   <xacro:if value="$(arg sim_ignition)">
-    <!-- Gazebo plugins -->
     <gazebo reference="world">
     </gazebo>
@@ -685,5 +486,5 @@
       <plugin filename="libign_ros2_control-system.so" name="ign_ros2_control::IgnitionROS2ControlPlugin">
         <parameters>$(arg simulation_controllers)</parameters>
-        <controller_manager_node_name>$(arg tf_prefix)controller_manager</controller_manager_node_name>
+        <controller_manager_node_name>controller_manager</controller_manager_node_name>
       </plugin>
     </gazebo>

File: UR5e/duo_ur/urdf/ur5e_macro.xacro (robot description, xacro)
@@ -53,5 +53,4 @@
     <xacro:if value="${generate_ros2_control_tag}">
       <!-- ros2 control include -->
-      <!-- <xacro:include filename="$(find duo_ur)/urdf/ur5e.ros2_control.xacro" /> -->
       <xacro:include filename="$(find duo_ur)/urdf/ur5e_prefixed.ros2_control.xacro" />
       <!-- ros2 control instance -->
