Commit message: Adjusted reference frame

File: UR5e/duo_ur/urdf/duo_ur_onehand.urdf.xacro (robot description, xacro)
@@ -72,5 +72,4 @@
    <xacro:property name="sensor_base_length" value="0.035"/>
    <xacro:property name="sensor_base_origin" value="0 0 0.03"/>
-   <link name="world" />
   <link name="mur">
     <visual>
@@ -89,9 +88,4 @@
     </collision>
   </link>
-  <joint name="world_to_mur" type="fixed">
-    <parent link="world"/>
-    <child link="mur"/>
-    <origin xyz="${mur_origin}"/>
-  </joint>
   <link name="hip">
     <visual>
