Commit message: Major clean up

File: UR5e/duo_ur/urdf/brainco_hand.urdf.xacro (robot description, xacro)
@@ -3,5 +3,5 @@
      Commit Version: 1.6.0-4-g7f85cfe  Build Version: 1.6.7995.38578
      For more information, please see http://wiki.ros.org/sw_urdf_exporter -->
-<robot xmlns:xacro="http://wiki.ros.org/xacro" name="BrainCoRightHandURDF">
+<robot xmlns:xacro="http://wiki.ros.org/xacro" name="brainco_hand">
   <xacro:macro name="brainco_hand" params="prefix:=''">
     <link name="${prefix}base_link">
@@ -14,14 +14,14 @@
         <origin xyz="0 0 0" rpy="0 0 0"/>
         <geometry>
-          <mesh filename="package://BrainCoRightHandURDF/meshes/base_link.STL"/>
-        </geometry>
-        <material name="">
-          <color rgba="0.75294 0.75294 0.75294 1"/>
-        </material>
-      </visual>
-      <collision>
-        <origin xyz="0 0 0" rpy="0 0 0"/>
-        <geometry>
-          <mesh filename="package://BrainCoRightHandURDF/meshes/base_link.STL"/>
+          <mesh filename="package://duo_ur/meshes/brainco/base_link.STL"/>
+        </geometry>
+        <material name="">
+          <color rgba="0.75294 0.75294 0.75294 1"/>
+        </material>
+      </visual>
+      <collision>
+        <origin xyz="0 0 0" rpy="0 0 0"/>
+        <geometry>
+          <mesh filename="package://duo_ur/meshes/brainco/base_link.STL"/>
         </geometry>
       </collision>
@@ -36,5 +36,5 @@
         <origin xyz="0 0 0" rpy="0 0 0"/>
         <geometry>
-          <mesh filename="package://BrainCoRightHandURDF/meshes/thumb_prox.STL"/>
+          <mesh filename="package://duo_ur/meshes/brainco/thumb_prox.STL"/>
         </geometry>
         <material name="">
@@ -45,5 +45,5 @@
         <origin xyz="0 0 0" rpy="0 0 0"/>
         <geometry>
-          <mesh filename="package://BrainCoRightHandURDF/meshes/thumb_prox.STL"/>
+          <mesh filename="package://duo_ur/meshes/brainco/thumb_prox.STL"/>
         </geometry>
       </collision>
@@ -63,14 +63,14 @@
         <origin xyz="0 0 0" rpy="0 0 0"/>
         <geometry>
-          <mesh filename="package://BrainCoRightHandURDF/meshes/thumb_dist.STL"/>
-        </geometry>
-        <material name="">
-          <color rgba="0.75294 0.75294 0.75294 1"/>
-        </material>
-      </visual>
-      <collision>
-        <origin xyz="0 0 0" rpy="0 0 0"/>
-        <geometry>
-          <mesh filename="package://BrainCoRightHandURDF/meshes/thumb_dist.STL"/>
+          <mesh filename="package://duo_ur/meshes/brainco/thumb_dist.STL"/>
+        </geometry>
+        <material name="">
+          <color rgba="0.75294 0.75294 0.75294 1"/>
+        </material>
+      </visual>
+      <collision>
+        <origin xyz="0 0 0" rpy="0 0 0"/>
+        <geometry>
+          <mesh filename="package://duo_ur/meshes/brainco/thumb_dist.STL"/>
         </geometry>
       </collision>
@@ -90,14 +90,14 @@
         <origin xyz="0 0 0" rpy="0 0 0"/>
         <geometry>
-          <mesh filename="package://BrainCoRightHandURDF/meshes/index_prox.STL"/>
-        </geometry>
-        <material name="">
-          <color rgba="0.75294 0.75294 0.75294 1"/>
-        </material>
-      </visual>
-      <collision>
-        <origin xyz="0 0 0" rpy="0 0 0"/>
-        <geometry>
-          <mesh filename="package://BrainCoRightHandURDF/meshes/index_prox.STL"/>
+          <mesh filename="package://duo_ur/meshes/brainco/index_prox.STL"/>
+        </geometry>
+        <material name="">
+          <color rgba="0.75294 0.75294 0.75294 1"/>
+        </material>
+      </visual>
+      <collision>
+        <origin xyz="0 0 0" rpy="0 0 0"/>
+        <geometry>
+          <mesh filename="package://duo_ur/meshes/brainco/index_prox.STL"/>
         </geometry>
       </collision>
@@ -117,14 +117,14 @@
         <origin xyz="0 0 0" rpy="0 0 0"/>
         <geometry>
-          <mesh filename="package://BrainCoRightHandURDF/meshes/index_dist.STL"/>
-        </geometry>
-        <material name="">
-          <color rgba="0.75294 0.75294 0.75294 1"/>
-        </material>
-      </visual>
-      <collision>
-        <origin xyz="0 0 0" rpy="0 0 0"/>
-        <geometry>
-          <mesh filename="package://BrainCoRightHandURDF/meshes/index_dist.STL"/>
+          <mesh filename="package://duo_ur/meshes/brainco/index_dist.STL"/>
+        </geometry>
+        <material name="">
+          <color rgba="0.75294 0.75294 0.75294 1"/>
+        </material>
+      </visual>
+      <collision>
+        <origin xyz="0 0 0" rpy="0 0 0"/>
+        <geometry>
+          <mesh filename="package://duo_ur/meshes/brainco/index_dist.STL"/>
         </geometry>
       </collision>
@@ -144,14 +144,14 @@
         <origin xyz="0 0 0" rpy="0 0 0"/>
         <geometry>
-          <mesh filename="package://BrainCoRightHandURDF/meshes/middle_prox.STL"/>
-        </geometry>
-        <material name="">
-          <color rgba="0.75294 0.75294 0.75294 1"/>
-        </material>
-      </visual>
-      <collision>
-        <origin xyz="0 0 0" rpy="0 0 0"/>
-        <geometry>
-          <mesh filename="package://BrainCoRightHandURDF/meshes/middle_prox.STL"/>
+          <mesh filename="package://duo_ur/meshes/brainco/middle_prox.STL"/>
+        </geometry>
+        <material name="">
+          <color rgba="0.75294 0.75294 0.75294 1"/>
+        </material>
+      </visual>
+      <collision>
+        <origin xyz="0 0 0" rpy="0 0 0"/>
+        <geometry>
+          <mesh filename="package://duo_ur/meshes/brainco/middle_prox.STL"/>
         </geometry>
       </collision>
@@ -171,14 +171,14 @@
         <origin xyz="0 0 0" rpy="0 0 0"/>
         <geometry>
-          <mesh filename="package://BrainCoRightHandURDF/meshes/middle_dist.STL"/>
-        </geometry>
-        <material name="">
-          <color rgba="0.75294 0.75294 0.75294 1"/>
-        </material>
-      </visual>
-      <collision>
-        <origin xyz="0 0 0" rpy="0 0 0"/>
-        <geometry>
-          <mesh filename="package://BrainCoRightHandURDF/meshes/middle_dist.STL"/>
+          <mesh filename="package://duo_ur/meshes/brainco/middle_dist.STL"/>
+        </geometry>
+        <material name="">
+          <color rgba="0.75294 0.75294 0.75294 1"/>
+        </material>
+      </visual>
+      <collision>
+        <origin xyz="0 0 0" rpy="0 0 0"/>
+        <geometry>
+          <mesh filename="package://duo_ur/meshes/brainco/middle_dist.STL"/>
         </geometry>
       </collision>
@@ -198,14 +198,14 @@
         <origin xyz="0 0 0" rpy="0 0 0"/>
         <geometry>
-          <mesh filename="package://BrainCoRightHandURDF/meshes/ring_prox.STL"/>
-        </geometry>
-        <material name="">
-          <color rgba="0.75294 0.75294 0.75294 1"/>
-        </material>
-      </visual>
-      <collision>
-        <origin xyz="0 0 0" rpy="0 0 0"/>
-        <geometry>
-          <mesh filename="package://BrainCoRightHandURDF/meshes/ring_prox.STL"/>
+          <mesh filename="package://duo_ur/meshes/brainco/ring_prox.STL"/>
+        </geometry>
+        <material name="">
+          <color rgba="0.75294 0.75294 0.75294 1"/>
+        </material>
+      </visual>
+      <collision>
+        <origin xyz="0 0 0" rpy="0 0 0"/>
+        <geometry>
+          <mesh filename="package://duo_ur/meshes/brainco/ring_prox.STL"/>
         </geometry>
       </collision>
@@ -225,14 +225,14 @@
         <origin xyz="0 0 0" rpy="0 0 0"/>
         <geometry>
-          <mesh filename="package://BrainCoRightHandURDF/meshes/ring_dist.STL"/>
-        </geometry>
-        <material name="">
-          <color rgba="0.75294 0.75294 0.75294 1"/>
-        </material>
-      </visual>
-      <collision>
-        <origin xyz="0 0 0" rpy="0 0 0"/>
-        <geometry>
-          <mesh filename="package://BrainCoRightHandURDF/meshes/ring_dist.STL"/>
+          <mesh filename="package://duo_ur/meshes/brainco/ring_dist.STL"/>
+        </geometry>
+        <material name="">
+          <color rgba="0.75294 0.75294 0.75294 1"/>
+        </material>
+      </visual>
+      <collision>
+        <origin xyz="0 0 0" rpy="0 0 0"/>
+        <geometry>
+          <mesh filename="package://duo_ur/meshes/brainco/ring_dist.STL"/>
         </geometry>
       </collision>
@@ -252,14 +252,14 @@
         <origin xyz="0 0 0" rpy="0 0 0"/>
         <geometry>
-          <mesh filename="package://BrainCoRightHandURDF/meshes/little_prox.STL"/>
-        </geometry>
-        <material name="">
-          <color rgba="0.75294 0.75294 0.75294 1"/>
-        </material>
-      </visual>
-      <collision>
-        <origin xyz="0 0 0" rpy="0 0 0"/>
-        <geometry>
-          <mesh filename="package://BrainCoRightHandURDF/meshes/little_prox.STL"/>
+          <mesh filename="package://duo_ur/meshes/brainco/little_prox.STL"/>
+        </geometry>
+        <material name="">
+          <color rgba="0.75294 0.75294 0.75294 1"/>
+        </material>
+      </visual>
+      <collision>
+        <origin xyz="0 0 0" rpy="0 0 0"/>
+        <geometry>
+          <mesh filename="package://duo_ur/meshes/brainco/little_prox.STL"/>
         </geometry>
       </collision>
@@ -279,14 +279,14 @@
         <origin xyz="0 0 0" rpy="0 0 0"/>
         <geometry>
-          <mesh filename="package://BrainCoRightHandURDF/meshes/little_dist.STL"/>
-        </geometry>
-        <material name="">
-          <color rgba="0.75294 0.75294 0.75294 1"/>
-        </material>
-      </visual>
-      <collision>
-        <origin xyz="0 0 0" rpy="0 0 0"/>
-        <geometry>
-          <mesh filename="package://BrainCoRightHandURDF/meshes/little_dist.STL"/>
+          <mesh filename="package://duo_ur/meshes/brainco/little_dist.STL"/>
+        </geometry>
+        <material name="">
+          <color rgba="0.75294 0.75294 0.75294 1"/>
+        </material>
+      </visual>
+      <collision>
+        <origin xyz="0 0 0" rpy="0 0 0"/>
+        <geometry>
+          <mesh filename="package://duo_ur/meshes/brainco/little_dist.STL"/>
         </geometry>
       </collision>

File: UR5e/duo_ur/urdf/duo_ur_onehand.urdf.xacro (robot description, xacro)
@@ -3,5 +3,5 @@
    <xacro:arg name="name" default="ur"/>
    <xacro:include filename="$(find duo_ur)/urdf/ur5e_macro.xacro"/>
-   <xacro:include filename="$(find BrainCoRightHandURDF)/urdf/BrainCoRightHandURDF.urdf.xacro"/>
+   <xacro:include filename="$(find duo_ur)/urdf/brainco_hand.urdf.xacro"/>
    <xacro:arg name="ur_type" default="ur5e"/>
    <xacro:arg name="tf_prefix_1" default="right_" />
@@ -43,5 +43,5 @@
    <xacro:arg name="sim_gazebo" default="false" />
    <xacro:arg name="sim_ignition" default="false" />
-   <xacro:arg name="simulation_controllers" default="$(find duo_ur)/config/duo_ur5e_controllers.yaml" />
+   <xacro:arg name="simulation_controllers" default="$(find duo_ur)/config/controllers.yaml" />
    <material name="Light_Grey">
     <color rgba="0.8 0.8 0.8 1.0"/>
